File: heimdall.sch (KiCad schematic (older format))
At the start: 13 parts, among them P1 CONN, Q1 Q_NMOS_DGS, U1 ESP-01, U2 TLP222A, U3 UA78M33CDCY

Commit message: Additional faffing, starting PCB
Parts:
- removed Q1: Q_NMOS_DGS, symbol Q_NMOS_DGS
- added R1: 680R, Resistors_SMD:R_0603, symbol R_Small
- C1, C2: footprint (none) -> Capacitors_SMD:C_0603
- D1, D3, D4: footprint (none) -> Diodes_SMD:SMA_Standard; Farnell (none) -> 1467636
- D2: footprint (none) -> Diodes_ThroughHole:Diode_DO-35_SOD27_Horizontal_RM10; Farnell (none) -> 2453723
- U2: footprint DIP-4 -> Housings_DIP:DIP-4_W7.62mm
- U3: footprint (none) -> TO_SOT_Packages_SMD:SOT-223
Changed lines of the file:
@@
 L ESP-01 U1
 U 1 1 57375DDB
-P 5150 1400
-F 0 "U1" H 5150 1150 60  0001 C CNN
-F 1 "ESP-01" H 5150 1650 60  0000 C CNN
-F 2 "Pin_Headers:Pin_Header_Straight_2x04" H 5150 1600 60  0001 C CNN
-F 3 "" H 5150 1600 60  0000 C CNN
-	1    5150 1400
+P 5300 1050
+F 0 "U1" H 5300 800 60  0001 C CNN
+F 1 "ESP-01" H 5300 1300 60  0000 C CNN
+F 2 "Pin_Headers:Pin_Header_Straight_2x04" H 5300 1250 60  0001 C CNN
+F 3 "" H 5300 1250 60  0000 C CNN
+	1    5300 1050
 	1    0    0    -1
 $EndComp
@@
 L GND #PWR01
 U 1 1 57375E64
-P 4650 1550
-F 0 "#PWR01" H 4650 1300 50  0001 C CNN
-F 1 "GND" H 4650 1400 50  0000 C CNN
-F 2 "" H 4650 1550 50  0000 C CNN
-F 3 "" H 4650 1550 50  0000 C CNN
-	1    4650 1550
+P 4800 1200
+F 0 "#PWR01" H 4800 950 50  0001 C CNN
+F 1 "GND" H 4800 1050 50  0000 C CNN
+F 2 "" H 4800 1200 50  0000 C CNN
+F 3 "" H 4800 1200 50  0000 C CNN
+	1    4800 1200
 	1    0    0    -1
 $EndComp
@@
 L +3.3V #PWR02
 U 1 1 57375E7A
-P 5650 1250
-F 0 "#PWR02" H 5650 1100 50  0001 C CNN
-F 1 "+3.3V" H 5650 1390 50  0000 C CNN
-F 2 "" H 5650 1250 50  0000 C CNN
-F 3 "" H 5650 1250 50  0000 C CNN
-	1    5650 1250
-	1    0    0    -1
-$EndComp
-NoConn ~ 5650 1350
-NoConn ~ 5650 1450
-NoConn ~ 5650 1550
-NoConn ~ 4650 1250
-NoConn ~ 4650 1450
-Text Label 4650 1350 2    60   ~ 0
+P 5800 900
+F 0 "#PWR02" H 5800 750 50  0001 C CNN
+F 1 "+3.3V" H 5800 1040 50  0000 C CNN
+F 2 "" H 5800 900 50  0000 C CNN
+F 3 "" H 5800 900 50  0000 C CNN
+	1    5800 900
+	1    0    0    -1
+$EndComp
+NoConn ~ 5800 1000
+NoConn ~ 5800 1100
+NoConn ~ 5800 1200
+NoConn ~ 4800 900
+NoConn ~ 4800 1100
+Text Label 4800 1000 2    60   ~ 0
 RELAY_TRIGGER
-$Comp
-L Q_NMOS_DGS Q1
-U 1 1 5738A49D
-P 3350 1200
-F 0 "Q1" H 3650 1250 50  0001 R CNN
-F 1 "Q_NMOS_DGS" H 4000 1150 50  0001 R CNN
-F 2 "" H 3550 1300 50  0000 C CNN
-F 3 "" H 3350 1200 50  0000 C CNN
-	1    3350 1200
-	1    0    0    -1
-$EndComp
-Text Label 3150 1200 2    60   ~ 0
+Text Label 3400 1600 2    60   ~ 0
 RELAY_TRIGGER
-Text Label 4050 800  0    60   ~ 0
+Text Label 4200 1600 0    60   ~ 0
 SW0
-Text Label 4050 1000 0    60   ~ 0
+Text Label 4200 1800 0    60   ~ 0
 SW1
 $Comp
 L GND #PWR03
 U 1 1 5738A554
-P 3450 1400
-F 0 "#PWR03" H 3450 1150 50  0001 C CNN
-F 1 "GND" H 3450 1250 50  0000 C CNN
-F 2 "" H 3450 1400 50  0000 C CNN
-F 3 "" H 3450 1400 50  0000 C CNN
-	1    3450 1400
+P 3600 1800
+F 0 "#PWR03" H 3600 1550 50  0001 C CNN
+F 1 "GND" H 3600 1650 50  0000 C CNN
+F 2 "" H 3600 1800 50  0000 C CNN
+F 3 "" H 3600 1800 50  0000 C CNN
+	1    3600 1800
 	1    0    0    -1
 $EndComp
@@
 L TLP222A U2
 U 1 1 5738A7E1
-P 3750 900
-F 0 "U2" H 3550 1100 50  0001 L CNN
-F 1 "TLP222A" H 3600 1100 50  0000 L CNN
-F 2 "DIP-4" H 3550 700 50  0001 L CIN
-F 3 "" H 3700 900 50  0000 L CNN
-	1    3750 900
-	1    0    0    -1
-$EndComp
-$Comp
-L +3.3V #PWR08
-U 1 1 5738A872
-P 3450 800
-F 0 "#PWR08" H 3450 650 50  0001 C CNN
-F 1 "+3.3V" H 3450 940 50  0000 C CNN
-F 2 "" H 3450 800 50  0000 C CNN
-F 3 "" H 3450 800 50  0000 C CNN
-	1    3450 800
+P 3900 1700
+F 0 "U2" H 3700 1900 50  0001 L CNN
+F 1 "TLP222A" H 3750 1900 50  0000 L CNN
+F 2 "Housings_DIP:DIP-4_W7.62mm" H 3700 1500 50  0001 L CIN
+F 3 "" H 3850 1700 50  0000 L CNN
+	1    3900 1700
 	1    0    0    -1
 $EndComp
@@
 F 0 "D2" H 1250 2330 50  0001 L CNN
 F 1 "D_Small" H 1150 2350 50  0001 L CNN
-F 2 "" V 1300 2250 50  0000 C CNN
+F 2 "Diodes_ThroughHole:Diode_DO-35_SOD27_Horizontal_RM10" V 1300 2250 50  0001 C CNN
 F 3 "" V 1300 2250 50  0000 C CNN
+F 4 "2453723" H 1300 2250 60  0001 C CNN "Farnell"
 	1    1300 2250
 	-1   0    0    -1
@@
 F 0 "D1" H 950 2420 50  0001 L CNN
 F 1 "TVS_Small" V 1000 2400 50  0001 L CNN
-F 2 "" V 1000 2450 50  0000 C CNN
+F 2 "Diodes_SMD:SMA_Standard" V 1000 2450 50  0001 C CNN
 F 3 "" V 1000 2350 50  0000 C CNN
+F 4 "1467636" H 1000 2350 60  0001 C CNN "Farnell"
 	1    1000 2350
 	0    1    1    0
 $EndComp
 $Comp
-L GND #PWR09
+L GND #PWR08
 U 1 1 5738AD57
 P 1100 2450
-F 0 "#PWR09" H 1100 2200 50  0001 C CNN
+F 0 "#PWR08" H 1100 2200 50  0001 C CNN
 F 1 "GND" H 1100 2300 50  0000 C CNN
 F 2 "" H 1100 2450 50  0000 C CNN
@@
 F 0 "D3" H 1700 920 50  0001 L CNN
 F 1 "TVS_Small" V 1750 900 50  0001 L CNN
-F 2 "" V 1750 950 50  0000 C CNN
+F 2 "Diodes_SMD:SMA_Standard" V 1750 950 50  0001 C CNN
 F 3 "" V 1750 850 50  0000 C CNN
+F 4 "1467636" H 1750 850 60  0001 C CNN "Farnell"
 	1    1750 850
 	0    1    1    0
@@
 Connection ~ 1750 750
 $Comp
-L GND #PWR010
+L GND #PWR09
 U 1 1 5738ADF2
 P 1750 950
-F 0 "#PWR010" H 1750 700 50  0001 C CNN
+F 0 "#PWR09" H 1750 700 50  0001 C CNN
 F 1 "GND" H 1750 800 50  0000 C CNN
 F 2 "" H 1750 950 50  0000 C CNN
@@
 F 0 "D4" H 1700 1420 50  0001 L CNN
 F 1 "TVS_Small" V 1750 1400 50  0001 L CNN
-F 2 "" V 1750 1450 50  0000 C CNN
+F 2 "Diodes_SMD:SMA_Standard" V 1750 1450 50  0001 C CNN
 F 3 "" V 1750 1350 50  0000 C CNN
+F 4 "1467636" H 1750 1350 60  0001 C CNN "Farnell"
 	1    1750 1350
 	0    1    1    0
@@
 Connection ~ 1750 1250
 $Comp
-L GND #PWR011
+L GND #PWR010
 U 1 1 5738AE0E
 P 1750 1450
-F 0 "#PWR011" H 1750 1200 50  0001 C CNN
+F 0 "#PWR010" H 1750 1200 50  0001 C CNN
 F 1 "GND" H 1750 1300 50  0000 C CNN
 F 2 "" H 1750 1450 50  0000 C CNN
@@
 F 0 "F1" H 1810 810 50  0001 L CNN
 F 1 "0.5A" H 1750 800 50  0000 L CNN
-F 2 "" H 1850 750 50  0000 C CNN
+F 2 "" H 1850 750 50  0001 C CNN
 F 3 "" H 1850 750 50  0000 C CNN
 	1    1850 750
@@
 F 0 "C1" H 1660 2420 50  0001 L CNN
 F 1 "0.33uF" H 1350 2250 50  0000 L CNN
-F 2 "" H 1650 2350 50  0000 C CNN
+F 2 "Capacitors_SMD:C_0603" H 1650 2350 50  0001 C CNN
 F 3 "" H 1650 2350 50  0000 C CNN
 	1    1650 2350
@@
 F 0 "C2" H 2560 2420 50  0001 L CNN
 F 1 "0.1uF" H 2560 2270 50  0000 L CNN
-F 2 "" H 2550 2350 50  0000 C CNN
+F 2 "Capacitors_SMD:C_0603" H 2550 2350 50  0001 C CNN
 F 3 "" H 2550 2350 50  0000 C CNN
 	1    2550 2350
@@
 F 0 "U3" H 2300 2100 60  0000 C CNN
 F 1 "UA78M33CDCY" H 2100 2450 60  0000 C CNN
-F 2 "" H 2180 2300 60  0000 C CNN
+F 2 "TO_SOT_Packages_SMD:SOT-223" H 2180 2300 60  0001 C CNN
 F 3 "" H 2180 2300 60  0000 C CNN
 F 4 "2296031" H 2100 2300 60  0001 C CNN "Farnell"
@@
 Connection ~ 2100 2650
 $Comp
-L GND #PWR012
+L GND #PWR011
 U 1 1 573A5BD7
 P 2100 2650
-F 0 "#PWR012" H 2100 2400 50  0001 C CNN
+F 0 "#PWR011" H 2100 2400 50  0001 C CNN
 F 1 "GND" H 2100 2500 50  0000 C CNN
 F 2 "" H 2100 2650 50  0000 C CNN
@@
 Connection ~ 1200 2250
 Connection ~ 1100 2450
+$Comp
+L R_Small R1
+U 1 1 573AE1A8
+P 3500 1600
+F 0 "R1" H 3530 1620 50  0001 L CNN
+F 1 "680R" V 3400 1500 50  0000 L CNN
+F 2 "Resistors_SMD:R_0603" H 3500 1600 50  0001 C CNN
+F 3 "" H 3500 1600 50  0000 C CNN
+	1    3500 1600
+	0    1    1    0
+$EndComp
 $EndSCHEMATC

Commit message: Updated some componants and shuffled PCB
Signed-off-by: Thomas Bytheway <tb403@cam.ac.uk>
Parts:
- added F2: 0.25A, Resistors_SMD:R_1206, symbol F_Small
- D1: footprint Diodes_SMD:SMA_Standard -> Resistors_SMD:R_0603; Farnell 1467636 -> 2368174
- D2: footprint Diodes_ThroughHole:Diode_DO-35_SOD27_Horizontal_RM10 -> Diodes_SMD:SOD-523; Farnell 2453723 -> 2453725
- D3, D4: Farnell 1467636 -> 1749308
- D5: value 30v -> 22v; footprint TO_SOT_Packages_SMD:SOT-23 -> Diodes_SMD:SOD-523; Farnell 2463495 -> 2285347
- F1: footprint (none) -> Resistors_SMD:R_1206; Farnell (none) -> 9921834
Connections:
- wire segments 8 -> 6
Changed lines of the file:
@@
 L D_Small D2
 U 1 1 5738AA45
-P 1300 2250
-F 0 "D2" H 1250 2330 50  0001 L CNN
-F 1 "D_Small" H 1150 2350 50  0001 L CNN
-F 2 "Diodes_ThroughHole:Diode_DO-35_SOD27_Horizontal_RM10" V 1300 2250 50  0001 C CNN
-F 3 "" V 1300 2250 50  0000 C CNN
-F 4 "2453723" H 1300 2250 60  0001 C CNN "Farnell"
-	1    1300 2250
+P 1550 2250
+F 0 "D2" H 1500 2330 50  0001 L CNN
+F 1 "D_Small" H 1400 2350 50  0001 L CNN
+F 2 "Diodes_SMD:SOD-523" V 1550 2250 50  0001 C CNN
+F 3 "" V 1550 2250 50  0000 C CNN
+F 4 "2453725" H 1550 2250 60  0001 C CNN "Farnell"
+	1    1550 2250
 	-1   0    0    -1
 $EndComp
@@
 L TVS_Small D1
 U 1 1 5738ACA8
-P 1000 2350
-F 0 "D1" H 950 2420 50  0001 L CNN
-F 1 "TVS_Small" V 1000 2400 50  0001 L CNN
-F 2 "Diodes_SMD:SMA_Standard" V 1000 2450 50  0001 C CNN
-F 3 "" V 1000 2350 50  0000 C CNN
-F 4 "1467636" H 1000 2350 60  0001 C CNN "Farnell"
-	1    1000 2350
+P 1250 2350
+F 0 "D1" H 1200 2420 50  0001 L CNN
+F 1 "TVS_Small" V 1250 2400 50  0001 L CNN
+F 2 "Resistors_SMD:R_0603" V 1250 2450 50  0001 C CNN
+F 3 "" V 1250 2350 50  0000 C CNN
+F 4 "2368174" H 1250 2350 60  0001 C CNN "Farnell"
+	1    1250 2350
 	0    1    1    0
 $EndComp
@@
 L GND #PWR08
 U 1 1 5738AD57
-P 1100 2450
-F 0 "#PWR08" H 1100 2200 50  0001 C CNN
-F 1 "GND" H 1100 2300 50  0000 C CNN
-F 2 "" H 1100 2450 50  0000 C CNN
-F 3 "" H 1100 2450 50  0000 C CNN
-	1    1100 2450
-	1    0    0    -1
-$EndComp
-Text Label 1000 2250 2    60   ~ 0
+P 1350 2450
+F 0 "#PWR08" H 1350 2200 50  0001 C CNN
+F 1 "GND" H 1350 2300 50  0000 C CNN
+F 2 "" H 1350 2450 50  0000 C CNN
+F 3 "" H 1350 2450 50  0000 C CNN
+	1    1350 2450
+	1    0    0    -1
+$EndComp
+Text Label 1250 2250 2    60   ~ 0
 VCC_IN
 Text Label 1750 750  2    60   ~ 0
@@
 F 2 "Diodes_SMD:SMA_Standard" V 1750 950 50  0001 C CNN
 F 3 "" V 1750 850 50  0000 C CNN
-F 4 "1467636" H 1750 850 60  0001 C CNN "Farnell"
+F 4 "1749308" H 1750 850 60  0001 C CNN "Farnell"
 	1    1750 850
 	0    1    1    0
@@
 F 2 "Diodes_SMD:SMA_Standard" V 1750 1450 50  0001 C CNN
 F 3 "" V 1750 1350 50  0000 C CNN
-F 4 "1467636" H 1750 1350 60  0001 C CNN "Farnell"
+F 4 "1749308" H 1750 1350 60  0001 C CNN "Farnell"
 	1    1750 1350
 	0    1    1    0
@@
 F 0 "F1" H 1810 810 50  0001 L CNN
 F 1 "0.5A" H 1750 800 50  0000 L CNN
-F 2 "" H 1850 750 50  0001 C CNN
+F 2 "Resistors_SMD:R_1206" H 1850 750 50  0001 C CNN
 F 3 "" H 1850 750 50  0000 C CNN
+F 4 "9921834" H 1850 750 60  0001 C CNN "Farnell"
 	1    1850 750
 	1    0    0    -1
 $EndComp
-Connection ~ 1000 2250
 Wire Wire Line
 	1750 1250 1800 1250
@@
 P 1650 2350
 F 0 "C1" H 1660 2420 50  0001 L CNN
-F 1 "0.33uF" H 1350 2250 50  0000 L CNN
+F 1 "0.33uF" V 1750 2150 50  0000 L CNN
 F 2 "Capacitors_SMD:C_0603" H 1650 2350 50  0001 C CNN
 F 3 "" H 1650 2350 50  0000 C CNN
@@
 	1    0    0    -1
 $EndComp
-Wire Wire Line
-	1400 2250 1650 2250
 $Comp
 L C_Small C2
@@
 L ZENERsmall D5
 U 1 1 573A5DEB
-P 1200 2350
-F 0 "D5" H 1200 2450 50  0001 C CNN
-F 1 "30v" V 1200 2450 50  0000 C CNN
-F 2 "TO_SOT_Packages_SMD:SOT-23" H 1200 2350 50  0001 C CNN
-F 3 "" H 1200 2350 50  0000 C CNN
-F 4 "2463495" H 1200 2350 60  0001 C CNN "Farnell"
-	1    1200 2350
-	0    1    1    0
-$EndComp
-Wire Wire Line
-	1200 2450 1000 2450
-Wire Wire Line
-	1000 2250 1200 2250
-Connection ~ 1200 2250
-Connection ~ 1100 2450
+P 1450 2350
+F 0 "D5" H 1450 2450 50  0001 C CNN
+F 1 "22v" V 1550 2450 50  0000 C CNN
+F 2 "Diodes_SMD:SOD-523" H 1450 2350 50  0001 C CNN
+F 3 "" H 1450 2350 50  0000 C CNN
+F 4 "2285347" H 1450 2350 60  0001 C CNN "Farnell"
+	1    1450 2350
+	0    1    1    0
+$EndComp
+Wire Wire Line
+	1450 2450 1250 2450
+Connection ~ 1350 2450
 $Comp
 L R_Small R1
@@
 	0    1    1    0
 $EndComp
+$Comp
+L F_Small F2
+U 1 1 573B1826
+P 1350 2250
+F 0 "F2" H 1310 2310 50  0001 L CNN
+F 1 "0.25A" H 1250 2300 50  0000 L CNN
+F 2 "Resistors_SMD:R_1206" H 1350 2250 50  0001 C CNN
+F 3 "" H 1350 2250 50  0000 C CNN
+F 4 "9921826" H 1350 2250 60  0001 C CNN "Farnell"
+	1    1350 2250
+	1    0    0    -1
+$EndComp
+Connection ~ 1450 2250
+Connection ~ 1250 2250
 $EndSCHEMATC

Commit message: Slight schematic faffing, more PCB juggling and sexification.
Parts:
- removed D2: D_Small, Diodes_SMD:SOD-523, symbol D_Small
- removed D5: 22v, Diodes_SMD:SOD-523, symbol ZENERsmall
- added C3, C4: 104, Capacitors_SMD:C_0603, symbol C_Small
- added C5: 226, Capacitors_SMD:C_1206, symbol C_Small
- C1: value 0.33uF -> 334; Farnell (none) -> 2496926
- C2: value 0.1uF -> 104; Farnell (none) -> 2496833
- U1: footprint Pin_Headers:Pin_Header_Straight_2x04 -> Socket_Strips:Socket_Strip_Straight_2x04
Connections:
- wire segments 6 -> 9
- no-connect marks 5 -> 4
Changed lines of the file:
@@
 F 0 "U1" H 5300 800 60  0001 C CNN
 F 1 "ESP-01" H 5300 1300 60  0000 C CNN
-F 2 "Pin_Headers:Pin_Header_Straight_2x04" H 5300 1250 60  0001 C CNN
+F 2 "Socket_Strips:Socket_Strip_Straight_2x04" H 5300 1250 60  0001 C CNN
 F 3 "" H 5300 1250 60  0000 C CNN
 	1    5300 1050
@@
 L +3.3V #PWR02
 U 1 1 57375E7A
-P 5800 900
-F 0 "#PWR02" H 5800 750 50  0001 C CNN
-F 1 "+3.3V" H 5800 1040 50  0000 C CNN
-F 2 "" H 5800 900 50  0000 C CNN
-F 3 "" H 5800 900 50  0000 C CNN
-	1    5800 900
-	1    0    0    -1
-$EndComp
-NoConn ~ 5800 1000
+P 6450 900
+F 0 "#PWR02" H 6450 750 50  0001 C CNN
+F 1 "+3.3V" H 6450 1040 50  0000 C CNN
+F 2 "" H 6450 900 50  0000 C CNN
+F 3 "" H 6450 900 50  0000 C CNN
+	1    6450 900
+	1    0    0    -1
+$EndComp
 NoConn ~ 5800 1100
 NoConn ~ 5800 1200
@@
 	1    0    0    -1
 $EndComp
-$Comp
-L D_Small D2
-U 1 1 5738AA45
-P 1550 2250
-F 0 "D2" H 1500 2330 50  0001 L CNN
-F 1 "D_Small" H 1400 2350 50  0001 L CNN
-F 2 "Diodes_SMD:SOD-523" V 1550 2250 50  0001 C CNN
-F 3 "" V 1550 2250 50  0000 C CNN
-F 4 "2453725" H 1550 2250 60  0001 C CNN "Farnell"
-	1    1550 2250
-	-1   0    0    -1
-$EndComp
 Text Label 950  750  0    60   ~ 0
 VCC_IN
@@
 L TVS_Small D1
 U 1 1 5738ACA8
-P 1250 2350
-F 0 "D1" H 1200 2420 50  0001 L CNN
-F 1 "TVS_Small" V 1250 2400 50  0001 L CNN
-F 2 "Resistors_SMD:R_0603" V 1250 2450 50  0001 C CNN
-F 3 "" V 1250 2350 50  0000 C CNN
-F 4 "2368174" H 1250 2350 60  0001 C CNN "Farnell"
-	1    1250 2350
+P 1450 2350
+F 0 "D1" H 1400 2420 50  0001 L CNN
+F 1 "TVS_Small" V 1450 2400 50  0001 L CNN
+F 2 "Resistors_SMD:R_0603" V 1450 2450 50  0001 C CNN
+F 3 "" V 1450 2350 50  0000 C CNN
+F 4 "2368174" H 1450 2350 60  0001 C CNN "Farnell"
+	1    1450 2350
 	0    1    1    0
 $EndComp
@@
 L GND #PWR08
 U 1 1 5738AD57
-P 1350 2450
-F 0 "#PWR08" H 1350 2200 50  0001 C CNN
-F 1 "GND" H 1350 2300 50  0000 C CNN
-F 2 "" H 1350 2450 50  0000 C CNN
-F 3 "" H 1350 2450 50  0000 C CNN
-	1    1350 2450
-	1    0    0    -1
-$EndComp
-Text Label 1250 2250 2    60   ~ 0
+P 1450 2450
+F 0 "#PWR08" H 1450 2200 50  0001 C CNN
+F 1 "GND" H 1450 2300 50  0000 C CNN
+F 2 "" H 1450 2450 50  0000 C CNN
+F 3 "" H 1450 2450 50  0000 C CNN
+	1    1450 2450
+	1    0    0    -1
+$EndComp
+Text Label 1450 2250 2    60   ~ 0
 VCC_IN
 Text Label 1750 750  2    60   ~ 0
@@
 P 1650 2350
 F 0 "C1" H 1660 2420 50  0001 L CNN
-F 1 "0.33uF" V 1750 2150 50  0000 L CNN
+F 1 "334" H 1670 2260 50  0000 L CNN
 F 2 "Capacitors_SMD:C_0603" H 1650 2350 50  0001 C CNN
 F 3 "" H 1650 2350 50  0000 C CNN
+F 4 "2496926" H 1650 2350 60  0001 C CNN "Farnell"
 	1    1650 2350
 	1    0    0    -1
@@
 P 2550 2350
 F 0 "C2" H 2560 2420 50  0001 L CNN
-F 1 "0.1uF" H 2560 2270 50  0000 L CNN
+F 1 "104" H 2560 2270 50  0000 L CNN
 F 2 "Capacitors_SMD:C_0603" H 2550 2350 50  0001 C CNN
 F 3 "" H 2550 2350 50  0000 C CNN
+F 4 "2496833" H 2550 2350 60  0001 C CNN "Farnell"
 	1    2550 2350
 	1    0    0    -1
@@
 Connection ~ 1650 2250
 Wire Wire Line
-	2550 2650 2550 2450
-Wire Wire Line
-	1650 2650 2550 2650
+	2550 2450 2550 2700
 Wire Wire Line
 	1650 2650 1650 2450
@@
 L GND #PWR011
 U 1 1 573A5BD7
-P 2100 2650
-F 0 "#PWR011" H 2100 2400 50  0001 C CNN
-F 1 "GND" H 2100 2500 50  0000 C CNN
-F 2 "" H 2100 2650 50  0000 C CNN
-F 3 "" H 2100 2650 50  0000 C CNN
-	1    2100 2650
-	1    0    0    -1
-$EndComp
-$Comp
-L ZENERsmall D5
-U 1 1 573A5DEB
-P 1450 2350
-F 0 "D5" H 1450 2450 50  0001 C CNN
-F 1 "22v" V 1550 2450 50  0000 C CNN
-F 2 "Diodes_SMD:SOD-523" H 1450 2350 50  0001 C CNN
-F 3 "" H 1450 2350 50  0000 C CNN
-F 4 "2285347" H 1450 2350 60  0001 C CNN "Farnell"
-	1    1450 2350
-	0    1    1    0
-$EndComp
-Wire Wire Line
-	1450 2450 1250 2450
-Connection ~ 1350 2450
+P 2100 2700
+F 0 "#PWR011" H 2100 2450 50  0001 C CNN
+F 1 "GND" H 2100 2550 50  0000 C CNN
+F 2 "" H 2100 2700 50  0000 C CNN
+F 3 "" H 2100 2700 50  0000 C CNN
+	1    2100 2700
+	1    0    0    -1
+$EndComp
 $Comp
 L R_Small R1
@@
 L F_Small F2
 U 1 1 573B1826
-P 1350 2250
-F 0 "F2" H 1310 2310 50  0001 L CNN
-F 1 "0.25A" H 1250 2300 50  0000 L CNN
-F 2 "Resistors_SMD:R_1206" H 1350 2250 50  0001 C CNN
-F 3 "" H 1350 2250 50  0000 C CNN
-F 4 "9921826" H 1350 2250 60  0001 C CNN "Farnell"
-	1    1350 2250
+P 1550 2250
+F 0 "F2" H 1510 2310 50  0001 L CNN
+F 1 "0.25A" H 1450 2300 50  0000 L CNN
+F 2 "Resistors_SMD:R_1206" H 1550 2250 50  0001 C CNN
+F 3 "" H 1550 2250 50  0000 C CNN
+F 4 "9921826" H 1550 2250 60  0001 C CNN "Farnell"
+	1    1550 2250
 	1    0    0    -1
 $EndComp
 Connection ~ 1450 2250
-Connection ~ 1250 2250
+Wire Wire Line
+	1650 2650 2100 2650
+Wire Wire Line
+	2100 2650 2100 2700
+Wire Wire Line
+	2100 2700 2550 2700
+Connection ~ 2100 2700
+$Comp
+L C_Small C3
+U 1 1 573BA384
+P 5900 1100
+F 0 "C3" H 5910 1170 50  0001 L CNN
+F 1 "104" H 5910 1020 50  0000 L CNN
+F 2 "Capacitors_SMD:C_0603" H 5900 1100 50  0001 C CNN
+F 3 "" H 5900 1100 50  0000 C CNN
+F 4 "2496833" H 5900 1100 60  0001 C CNN "Farnell"
+	1    5900 1100
+	1    0    0    -1
+$EndComp
+$Comp
+L C_Small C4
+U 1 1 573BA392
+P 6150 1000
+F 0 "C4" H 6160 1070 50  0001 L CNN
+F 1 "104" H 6160 920 50  0000 L CNN
+F 2 "Capacitors_SMD:C_0603" H 6150 1000 50  0001 C CNN
+F 3 "" H 6150 1000 50  0000 C CNN
+F 4 "2496833" H 6150 1000 60  0001 C CNN "Farnell"
+	1    6150 1000
+	1    0    0    -1
+$EndComp
+$Comp
+L C_Small C5
+U 1 1 573BA3A0
+P 6450 1000
+F 0 "C5" H 6460 1070 50  0001 L CNN
+F 1 "226" H 6460 920 50  0000 L CNN
+F 2 "Capacitors_SMD:C_1206" H 6450 1000 50  0001 C CNN
+F 3 "" H 6450 1000 50  0000 C CNN
+F 4 "2497155" H 6450 1000 60  0001 C CNN "Farnell"
+	1    6450 1000
+	1    0    0    -1
+$EndComp
+Wire Wire Line
+	5800 1000 5900 1000
+Wire Wire Line
+	5800 900  6450 900
+Connection ~ 6150 900
+Connection ~ 6450 900
+$Comp
+L GND #PWR012
+U 1 1 573BA3FE
+P 5900 1200
+F 0 "#PWR012" H 5900 950 50  0001 C CNN
+F 1 "GND" H 5900 1050 50  0000 C CNN
+F 2 "" H 5900 1200 50  0000 C CNN
+F 3 "" H 5900 1200 50  0000 C CNN
+	1    5900 1200
+	1    0    0    -1
+$EndComp
+$Comp
+L GND #PWR013
+U 1 1 573BA40C
+P 6150 1100
+F 0 "#PWR013" H 6150 850 50  0001 C CNN
+F 1 "GND" H 6150 950 50  0000 C CNN
+F 2 "" H 6150 1100 50  0000 C CNN
+F 3 "" H 6150 1100 50  0000 C CNN
+	1    6150 1100
+	1    0    0    -1
+$EndComp
+$Comp
+L GND #PWR014
+U 1 1 573BA41A
+P 6450 1100
+F 0 "#PWR014" H 6450 850 50  0001 C CNN
+F 1 "GND" H 6450 950 50  0000 C CNN
+F 2 "" H 6450 1100 50  0000 C CNN
+F 3 "" H 6450 1100 50  0000 C CNN
+	1    6450 1100
+	1    0    0    -1
+$EndComp
 $EndSCHEMATC

Commit message: Much faffing, many switch mode supply, very PCB.
Parts:
- removed U3: UA78M33CDCY, TO_SOT_Packages_SMD:SOT-223, symbol UA78M33CDCY
- added C6: 2u2, Capacitors_SMD:C_0603, symbol C_Small
- added L1: 10u, Wurth:WE-TPC, symbol L_Small
- added Q1: FDN304P, Housings_SSOT:SuperSOT-3, symbol Q_PMOS_GDS
- added R2: 100K, Resistors_SMD:R_0603, symbol R_Small
- added R3: 1K, Resistors_SMD:R_0603, symbol R_Small
- added U3: TPS62177, Housing_WSON:WSON-10, symbol TPS62177
- C1: value 334 -> 22u; Farnell 2496926 -> 2496833
- C2, C3, C4: value 104 -> 100n
- C5: value 226 -> 22u; footprint Capacitors_SMD:C_1206 -> Capacitors_SMD:C_0603
- F2: value 0.25A -> 0.5A; Farnell 9921826 -> 9921834
- R1: footprint Resistors_SMD:R_0603 -> Resistors_SMD:R_1206
- U1: footprint Socket_Strips:Socket_Strip_Straight_2x04 -> esp:ESP-01-NoSilk
Connections:
- net +3V3: now also C1.1, L1.2, Q1.3 (S), R2.2, U3.10 (VOS), U3.8 (SLEEP); no longer C2.1, C4.1, C5.1, U1.8 (VCC)
- net GND: now also C6.2, U3.1 (PGND), U3.11 (ETP), U3.5 (FB), U3.6 (AGND); no longer C2.2
- net at U1.4 (CH_PD): now also C4.1, C5.1, F2.1, U1.8 (VCC)
- net PWROUT: now reaches F2.2
- net PWROUT: now also C2.1, Q1.2 (D); no longer C1.1
- net VCC_IN renamed VCC
- net VCC: now also C6.1, U3.2 (VIN), U3.3 (EN); no longer F2.1
- new net: L1.1, U3.9 (SW)
- new net: C2.2, Q1.1 (G), R3.2
- new net PG: R2.1, R3.1, U3.7 (PG)
- no-connect marks 4 -> 3

Commit message: Various shuffling
Parts:
- R1: footprint Resistors_SMD:R_1206 -> Resistors_SMD:R_0603
Changed lines of the file:
@@
 F 0 "R1" H 3180 970 50  0001 L CNN
 F 1 "680R" V 3050 850 50  0000 L CNN
-F 2 "Resistors_SMD:R_1206" H 3150 950 50  0001 C CNN
+F 2 "Resistors_SMD:R_0603" H 3150 950 50  0001 C CNN
 F 3 "" H 3150 950 50  0000 C CNN
 	1    3150 950

Commit message: More faffing
Changed lines of the file:
@@
 P 6500 750
 F 0 "#FLG?" H 6500 845 50  0001 C CNN
-F 1 "PWR_FLAG" V 6500 928 50  0000 L CNN
+F 1 "PWR_FLAG" H 6500 950 50  0000 L CNN
 F 2 "" H 6500 750 50  0000 C CNN
 F 3 "" H 6500 750 50  0000 C CNN

Commit message: PMOS NMOS fun
Parts:
- removed Q1: FDN304P, Housings_SSOT:SuperSOT-3, symbol Q_PMOS_GDS
- added Q1: FDN337N, Housings_SSOT:SuperSOT-3, symbol Q_NMOS_GDS
Connections:
- net +3V3: now also Q1.2 (D)
- net PWROUT: now also Q1.3 (S)
- net at C2.2, R3.2: now also Q1.1 (G)
Changed lines of the file:
@@
 	2900 2800 2950 2800
 $Comp
-L Q_PMOS_GDS Q1
-U 1 1 57583146
-P 4300 1900
-F 0 "Q1" V 4628 1900 50  0001 C CNN
-F 1 "FDN304P" V 4500 2000 50  0000 C CNN
-F 2 "Housings_SSOT:SuperSOT-3" H 4500 2000 50  0001 C CNN
-F 3 "http://www.farnell.com/datasheets/238539.pdf" H 4300 1900 50  0001 C CNN
-F 4 "9846298" V 4300 1900 60  0001 C CNN "Farnell"
-	1    4300 1900
-	0    1    -1   0
-$EndComp
-$Comp
-L PWR_FLAG #FLG?
+L PWR_FLAG #FLG021
 U 1 1 57585735
 P 6500 750
-F 0 "#FLG?" H 6500 845 50  0001 C CNN
+F 0 "#FLG021" H 6500 845 50  0001 C CNN
 F 1 "PWR_FLAG" H 6500 950 50  0000 L CNN
 F 2 "" H 6500 750 50  0000 C CNN
@@
 Wire Wire Line
 	6800 750  6700 750
+$Comp
+L Q_NMOS_GDS Q1
+U 1 1 575976FE
+P 4300 1900
+F 0 "Q1" V 4536 1900 50  0001 C CNN
+F 1 "FDN337N" V 4500 1800 50  0000 C CNN
+F 2 "Housings_SSOT:SuperSOT-3" V 4537 1900 50  0001 C CNN
+F 3 "http://www.farnell.com/datasheets/220571.pdf" V 4537 1900 50  0001 C CNN
+F 4 "9845356" V 4300 1900 60  0001 C CNN "Farnell"
+	1    4300 1900
+	0    -1   -1   0
+$EndComp
 $EndSCHEMATC
